Commit message: Info update

File: description/robot_core.xacro (robot description, xacro)
@@ -2,4 +2,5 @@
 <robot xmlns:xacro="http://www.ros.org/wiki/xacro"  >
     <xacro:include filename="inertial_macros.xacro"/>
+<!--MATERIALS-->
     <material name="white">
         <color rgba="1 1 1 1" />
@@ -42,12 +43,12 @@
         </xacro:inertial_box>
     </link>
-<!--LEFT WHEEL LINK-->
-    <joint name ="left_wheel_joint" type="continuous">
+<!--FRONT LEFT WHEEL LINK-->
+    <joint name ="front_left_wheel_joint" type="continuous">
         <parent link="base_link"/>
-        <child link="left_wheel"/>
-        <origin xyz="0 0.100 0" rpy="-${pi/2} 0 0"/>
+        <child link="front_left_wheel"/>
+        <origin xyz="-0.075 0.100 0" rpy="-${pi/2} 0 0"/>
         <axis xyz="0 0 1"/>
     </joint>
-    <link name="left_wheel">
+    <link name="front_left_wheel">
         <visual>
             <geometry>
@@ -66,12 +67,108 @@
         </xacro:inertial_cylinder>
     </link>
-<!--RIGHT WHEEL LINK-->
-    <joint name ="right_wheel_joint" type="continuous">
+<!--FRONT RIGHT WHEEL LINK-->
+    <joint name ="front_right_wheel_joint" type="continuous">
         <parent link="base_link"/>
-        <child link="right_wheel"/>
+        <child link="front_right_wheel"/>
+        <origin xyz="-0.075 -0.100 0" rpy="${pi/2} 0 0"/>
+        <axis xyz="0 0 -1"/>
+    </joint>
+    <link name="front_right_wheel">
+        <visual>
+            <geometry>
+                <cylinder length="0.030" radius="0.030"/>
+            </geometry>
+            <material name ="black"/>
+        </visual>
+        <collision>
+            <geometry>
+                <cylinder length="0.030" radius="0.030"/>
+            </geometry>
+            <material name ="black"/>
+        </collision>
+        <xacro:inertial_cylinder mass="0.1" length="0.03" radius="0.03">
+            <origin xyz="0 0 0" rpy="0 0 0"/>
+        </xacro:inertial_cylinder>
+    </link>
+    <!--MIDDLE LEFT WHEEL LINK-->
+    <joint name ="middle_left_wheel_joint" type="continuous">
+        <parent link="base_link"/>
+        <child link="middle_left_wheel"/>
+        <origin xyz="0 0.100 0" rpy="-${pi/2} 0 0"/>
+        <axis xyz="0 0 1"/>
+    </joint>
+    <link name="middle_left_wheel">
+        <visual>
+            <geometry>
+                <cylinder length="0.03" radius="0.03"/>
+            </geometry>
+            <material name="black"/>
+        </visual>
+        <collision>
+            <geometry>
+                <cylinder length="0.030" radius="0.030"/>
+            </geometry>
+            <material name="black"/>
+        </collision>
+        <xacro:inertial_cylinder mass="0.1" length="0.03" radius="0.03">
+            <origin xyz="0 0 0" rpy="0 0 0"/>
+        </xacro:inertial_cylinder>
+    </link>
+<!--MIDDLE RIGHT WHEEL LINK-->
+    <joint name ="middle_right_wheel_joint" type="continuous">
+        <parent link="base_link"/>
+        <child link="middle_right_wheel"/>
         <origin xyz="0 -0.100 0" rpy="${pi/2} 0 0"/>
         <axis xyz="0 0 -1"/>
     </joint>
-    <link name="right_wheel">
+    <link name="middle_right_wheel">
+        <visual>
+            <geometry>
+                <cylinder length="0.030" radius="0.030"/>
+            </geometry>
+            <material name ="black"/>
+        </visual>
+        <collision>
+            <geometry>
+                <cylinder length="0.030" radius="0.030"/>
+            </geometry>
+            <material name ="black"/>
+        </collision>
+        <xacro:inertial_cylinder mass="0.1" length="0.03" radius="0.03">
+            <origin xyz="0 0 0" rpy="0 0 0"/>
+        </xacro:inertial_cylinder>
+    </link>
+    <!--BACK LEFT WHEEL LINK-->
+    <joint name ="back_left_wheel_joint" type="continuous">
+        <parent link="base_link"/>
+        <child link="back_left_wheel"/>
+        <origin xyz="0.065 0.100 0" rpy="-${pi/2} 0 0"/>
+        <axis xyz="0 0 1"/>
+    </joint>
+    <link name="back_left_wheel">
+        <visual>
+            <geometry>
+                <cylinder length="0.03" radius="0.03"/>
+            </geometry>
+            <material name="black"/>
+        </visual>
+        <collision>
+            <geometry>
+                <cylinder length="0.030" radius="0.030"/>
+            </geometry>
+            <material name="black"/>
+        </collision>
+        <xacro:inertial_cylinder mass="0.1" length="0.03" radius="0.03">
+            <origin xyz="0 0 0" rpy="0 0 0"/>
+        </xacro:inertial_cylinder>
+    </link>
+<!--BACK RIGHT WHEEL LINK-->
+    <joint name ="back_right_wheel_joint" type="continuous">
+        <parent link="base_link"/>
+        <child link="back_right_wheel"/>
+        <origin xyz="0.065 -0.100 0" rpy="${pi/2} 0 0"/>
+        <axis xyz="0 0 -1"/>
+    </joint>
+    <link name="back_right_wheel">
         <visual>
             <geometry>

Commit message: First working simulation robot

File: description/robot_core.xacro (robot description, xacro)
@@ -43,6 +43,63 @@
         </xacro:inertial_box>
     </link>
+    <gazebo reference="chassis">
+        <material>Gazebo/White</material>
+    </gazebo>
+<!--BACK LEFT WHEEL LINK-->
+    <joint name ="back_left_wheel_joint" type="continuous">
+        <parent link="base_link"/>
+        <child link="back_left_wheel"/>
+        <origin xyz="0.065 0.100 0" rpy="-${pi/2} 0 0"/>
+        <axis xyz="0 0 1"/>
+    </joint>
+    <link name="back_left_wheel">
+        <visual>
+            <geometry>
+                <cylinder length="0.03" radius="0.03"/>
+            </geometry>
+            <material name="black"/>
+        </visual>
+        <collision>
+            <geometry>
+                <cylinder length="0.030" radius="0.030"/>
+            </geometry>
+            <material name="black"/>
+        </collision>
+        <xacro:inertial_cylinder mass="0.1" length="0.03" radius="0.03">
+            <origin xyz="0 0 0" rpy="0 0 0"/>
+        </xacro:inertial_cylinder>
+    </link>
+    <gazebo reference="back_left_wheel">
+        <material>Gazebo/Black</material>
+    </gazebo>
+<!--BACK RIGHT WHEEL LINK-->
+    <joint name ="back_right_wheel_joint" type="continuous">
+        <parent link="base_link"/>
+        <child link="back_right_wheel"/>
+        <origin xyz="0.065 -0.100 0" rpy="${pi/2} 0 0"/>
+        <axis xyz="0 0 -1"/>
+    </joint>
+    <link name="back_right_wheel">
+        <visual>
+            <geometry>
+                <cylinder length="0.030" radius="0.030"/>
+            </geometry>
+            <material name ="black"/>
+        </visual>
+        <collision>
+            <geometry>
+                <cylinder length="0.030" radius="0.030"/>
+            </geometry>
+            <material name ="black"/>
+        </collision>
+        <xacro:inertial_cylinder mass="0.1" length="0.03" radius="0.03">
+            <origin xyz="0 0 0" rpy="0 0 0"/>
+        </xacro:inertial_cylinder>
+    </link>
+    <gazebo reference="back_right_wheel">
+        <material>Gazebo/Black</material>
+    </gazebo>
 <!--FRONT LEFT WHEEL LINK-->
-    <joint name ="front_left_wheel_joint" type="continuous">
+    <joint name ="front_left_wheel_joint" type="fixed">
         <parent link="base_link"/>
         <child link="front_left_wheel"/>
@@ -67,6 +124,11 @@
         </xacro:inertial_cylinder>
     </link>
+    <gazebo reference="front_left_wheel">
+        <material>Gazebo/Black</material>
+        <mu1 value="0.001"/>
+        <mu2 value="0.001"/>
+    </gazebo>
 <!--FRONT RIGHT WHEEL LINK-->
-    <joint name ="front_right_wheel_joint" type="continuous">
+    <joint name ="front_right_wheel_joint" type="fixed">
         <parent link="base_link"/>
         <child link="front_right_wheel"/>
@@ -91,6 +153,11 @@
         </xacro:inertial_cylinder>
     </link>
-    <!--MIDDLE LEFT WHEEL LINK-->
-    <joint name ="middle_left_wheel_joint" type="continuous">
+    <gazebo reference="front_right_wheel">
+        <material>Gazebo/Black</material>
+        <mu1 value="0.001"/>
+        <mu2 value="0.001"/>
+    </gazebo>
+<!--MIDDLE LEFT WHEEL LINK-->
+    <joint name ="middle_left_wheel_joint" type="fixed">
         <parent link="base_link"/>
         <child link="middle_left_wheel"/>
@@ -115,6 +182,11 @@
         </xacro:inertial_cylinder>
     </link>
+    <gazebo reference="middle_left_wheel">
+        <material>Gazebo/Black</material>
+        <mu1 value="0.001"/>
+        <mu2 value="0.001"/>
+    </gazebo>
 <!--MIDDLE RIGHT WHEEL LINK-->
-    <joint name ="middle_right_wheel_joint" type="continuous">
+    <joint name ="middle_right_wheel_joint" type="fixed">
         <parent link="base_link"/>
         <child link="middle_right_wheel"/>
@@ -139,51 +211,8 @@
         </xacro:inertial_cylinder>
     </link>
-    <!--BACK LEFT WHEEL LINK-->
-    <joint name ="back_left_wheel_joint" type="continuous">
-        <parent link="base_link"/>
-        <child link="back_left_wheel"/>
-        <origin xyz="0.065 0.100 0" rpy="-${pi/2} 0 0"/>
-        <axis xyz="0 0 1"/>
-    </joint>
-    <link name="back_left_wheel">
-        <visual>
-            <geometry>
-                <cylinder length="0.03" radius="0.03"/>
-            </geometry>
-            <material name="black"/>
-        </visual>
-        <collision>
-            <geometry>
-                <cylinder length="0.030" radius="0.030"/>
-            </geometry>
-            <material name="black"/>
-        </collision>
-        <xacro:inertial_cylinder mass="0.1" length="0.03" radius="0.03">
-            <origin xyz="0 0 0" rpy="0 0 0"/>
-        </xacro:inertial_cylinder>
-    </link>
-<!--BACK RIGHT WHEEL LINK-->
-    <joint name ="back_right_wheel_joint" type="continuous">
-        <parent link="base_link"/>
-        <child link="back_right_wheel"/>
-        <origin xyz="0.065 -0.100 0" rpy="${pi/2} 0 0"/>
-        <axis xyz="0 0 -1"/>
-    </joint>
-    <link name="back_right_wheel">
-        <visual>
-            <geometry>
-                <cylinder length="0.030" radius="0.030"/>
-            </geometry>
-            <material name ="black"/>
-        </visual>
-        <collision>
-            <geometry>
-                <cylinder length="0.030" radius="0.030"/>
-            </geometry>
-            <material name ="black"/>
-        </collision>
-        <xacro:inertial_cylinder mass="0.1" length="0.03" radius="0.03">
-            <origin xyz="0 0 0" rpy="0 0 0"/>
-        </xacro:inertial_cylinder>
-    </link>
+    <gazebo reference="middle_right_wheel">
+        <material>Gazebo/Black</material>
+        <mu1 value="0.001"/>
+        <mu2 value="0.001"/>
+    </gazebo>
 </robot>
